File: mote-hardware/rp2354.kicad_sch (KiCad schematic)
At the start: 41 parts, among them J4 SM03B-SRSS-TB, J5 Conn_01x03_Pin, J6 Conn_01x03_Pin, SW1 SW_Push, SW2 SW_Push, U1 RP2354_60QFN, U4 RP Radio Module 2, Y1 ABM8-272-T3

Commit message: mote-hardware v0.2.0 (#63)
Improvements to the pcb design for rev v0.2.0
Parts:
- removed D18, D19, D20, D21, D22, D23: PTVS5V0S1UR-FS, Diode_SMD:D_SOD-123, symbol Diode:PTVS5V0Z1USK
- added U13, U6, U7: TPD2E2U06DCK, Package_TO_SOT_SMD:SOT-323_SC-70, symbol Power_Protection:TPD2E2U06DCK
- H5, H6: footprint MountingHole:MountingHole_4.3mm_M4_DIN965_Pad_TopOnly -> mote-hardware:MountingHole_4.3mm_M4_DIN965_Pad_TopOnly
Connections:
- net GND: now also U13.3, U6.3, U7.3
- net RUN: now also U13.1
- net SWCLK: now also U6.1
- net SWD: now also U6.2
- net UART0_RX: now also U7.1
- net UART0_TX: now also U7.2
- net ~{USB_BOOT}: now also U13.2
Other:
- company: github.com/empriselab/mote-core -> github.com/empriselab/mote
- moved on the sheet: J4, J5, J6
