File: mote-hardware/rp2354.kicad_sch (KiCad schematic)
At the start: 41 parts, among them J4 SM03B-SRSS-TB, J5 Conn_01x03_Pin, J6 Conn_01x03_Pin, SW1 SW_Push, SW2 SW_Push, U1 RP2354_60QFN, U4 RP Radio Module 2, Y1 ABM8-272-T3

Commit message: Include tail mount nuts in BOM
Parts:
- H5, H6: footprint MountingHole:MountingHole_4.3mm_M4_DIN965_Pad_TopOnly -> mote-hardware:MountingHole_4.3mm_M4_DIN965_Pad_TopOnly
Changed lines of the file:
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@@
 			)
 		)
-		(property "Footprint" "MountingHole:MountingHole_4.3mm_M4_DIN965_Pad_TopOnly"
+		(property "Footprint" "mote-hardware:MountingHole_4.3mm_M4_DIN965_Pad_TopOnly"
 			(at 265.43 262.89 0)
 			(effects
@@
 			)
 		)
-		(property "Footprint" "MountingHole:MountingHole_4.3mm_M4_DIN965_Pad_TopOnly"
+		(property "Footprint" "mote-hardware:MountingHole_4.3mm_M4_DIN965_Pad_TopOnly"
 			(at 275.59 270.51 0)
 			(effects

Commit message: Update schematic with low cap / high speed TVS diodes
Parts:
- removed D18, D19, D20, D21, D22, D23: PTVS5V0S1UR-FS, Diode_SMD:D_SOD-123, symbol Diode:PTVS5V0Z1USK
- added U13, U6, U7: TPD2E2U06DCK, Package_TO_SOT_SMD:SOT-323_SC-70, symbol Power_Protection:TPD2E2U06DCK
Connections:
- net GND: now also U13.3, U6.3, U7.3
- net RUN: now also U13.1
- net SWCLK: now also U6.1
- net SWD: now also U6.2
- net UART0_RX: now also U7.1
- net UART0_TX: now also U7.2
- net ~{USB_BOOT}: now also U13.2
Other:
- moved on the sheet: J4, J5, J6

Commit message: Layout for new tvs diodes
Other:
- company: github.com/empriselab/mote-core -> github.com/empriselab/mote
Changed lines of the file:
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@@
 	(title_block
 		(title "Mote")
-		(date "2026-04-25")
-		(rev "V0.1.0")
-		(company "github.com/empriselab/mote-core")
+		(date "2026-05-25")
+		(rev "V0.2.0")
+		(company "github.com/empriselab/mote")
 	)
 	(circle

Commit message: Update postition and rotation values for new components (#69)
Parts:
- U13, U6, U7: JLCPCB_CORRECTION 0; 0; 0 -> 0; 0; -90
- U4: JLCPCB_CORRECTION 0; 0; 0 -> 0;2.512; 0
- Y1: JLCPCB_CORRECTION 0; 0; 0 -> 0;0; 0
Changed lines of the file:
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@@
 			)
 		)
-		(property "JLCPCB_CORRECTION" "0; 0; 0"
+		(property "JLCPCB_CORRECTION" "0; 0; -90"
 			(at 383.54 210.82 0)
 			(effects
@@
 			)
 		)
-		(property "JLCPCB_CORRECTION" "0; 0; 0"
+		(property "JLCPCB_CORRECTION" "0;2.512; 0"
 			(at 336.55 116.84 0)
 			(effects
@@
 			)
 		)
-		(property "JLCPCB_CORRECTION" "0; 0; 0"
+		(property "JLCPCB_CORRECTION" "0;0; 0"
 			(at 328.93 43.18 90)
 			(effects
@@
 			)
 		)
-		(property "JLCPCB_CORRECTION" "0; 0; 0"
+		(property "JLCPCB_CORRECTION" "0; 0; -90"
 			(at 383.54 233.68 0)
 			(effects
@@
 			)
 		)
-		(property "JLCPCB_CORRECTION" "0; 0; 0"
+		(property "JLCPCB_CORRECTION" "0; 0; -90"
 			(at 50.8 171.45 0)
 			(effects
