File: mote-hardware/mote-hardware.kicad_sch (KiCad schematic)
At the start: 0 parts

Commit message: mote-hardware v0.2.0 (#63)
Improvements to the pcb design for rev v0.2.0
Other:
- company: github.com/empriselab/mote-core -> github.com/empriselab/mote
Changed lines of the file:
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@@
 	(title_block
 		(title "Mote")
-		(date "2026-04-25")
-		(rev "V0.1.0")
-		(company "github.com/empriselab/mote-core")
+		(date "2026-05-25")
+		(rev "V0.2.0")
+		(company "github.com/empriselab/mote")
 	)
 	(text "Mote Top-Level Design"

Commit message: Small tweaks and fixes to the schematic (#68)
Other:
- sheet lidar ports: added lidar_rx, lidar_tx; removed RX, TX
- sheet status leds ports: added LED_RX; removed rx
Changed lines of the file:
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@@
 	(title_block
 		(title "Mote")
-		(date "2026-05-25")
+		(date "2026-06-07")
 		(rev "V0.2.0")
 		(company "github.com/empriselab/mote")
@@
 			)
 		)
-		(pin "RX" input
-			(at 205.74 104.14 180)
-			(effects
-				(font
-					(size 1.27 1.27)
-				)
-				(justify left)
-			)
-		)
 		(pin "GND" passive
 			(at 205.74 107.95 180)
@@
 			)
 		)
-		(pin "TX" output
-			(at 205.74 101.6 180)
-			(effects
-				(font
-					(size 1.27 1.27)
-				)
-				(justify left)
-			)
-		)
 		(pin "+5v" passive
 			(at 205.74 96.52 180)
+			(effects
+				(font
+					(size 1.27 1.27)
+				)
+				(justify left)
+			)
+		)
+		(pin "lidar_rx" input
+			(at 205.74 104.14 180)
+			(effects
+				(font
+					(size 1.27 1.27)
+				)
+				(justify left)
+			)
+		)
+		(pin "lidar_tx" output
+			(at 205.74 101.6 180)
 			(effects
 				(font
@@
 			)
 		)
-		(pin "GND" passive
-			(at 76.2 72.39 0)
-			(effects
-				(font
-					(size 1.27 1.27)
-				)
-				(justify right)
-			)
-		)
 		(pin "+3v3" passive
 			(at 76.2 53.34 0)
@@
 		(pin "CC1" output
 			(at 76.2 64.77 0)
+			(effects
+				(font
+					(size 1.27 1.27)
+				)
+				(justify right)
+			)
+		)
+		(pin "GND" input
+			(at 76.2 72.39 0)
 			(effects
 				(font
@@
 			)
 		)
-		(pin "rx" input
-			(at 205.74 148.59 180)
-			(effects
-				(font
-					(size 1.27 1.27)
-				)
-				(justify left)
-			)
-		)
 		(pin "+3v3" passive
 			(at 205.74 144.78 180)
 			(effects
 				(font
+					(size 1.27 1.27)
+				)
+				(justify left)
+			)
+		)
+		(pin "LED_RX" input
+			(at 205.74 148.59 180)
+			(effects
+				(font
